File: Fanstel-kicad-library.sch (KiCad schematic (older format))
At the start: 7 parts, among them U1 BC832-V0, U2 BT832L, U3 BC832-V1, U4 BM832, U5 BT832X, U6 BM840, U7 BT840

Commit message: Fixed issue #1
Parts:
- removed U1: BC832-V0, Fanstel_modules:BC832-BC832, symbol BC832-V0
- removed U2: BT832L, Fanstel_modules:BT832-BT832L, symbol BT832L
- removed U3: BC832-V1, Fanstel_modules:BC832-BC832, symbol BC832-V1
- removed U4: BM832, Fanstel_modules:BM832-1-BM832, symbol BM832
- removed U5: BT832X, Fanstel_modules:BT832X-BT832X, symbol BT832X
- removed U6: BM840, Fanstel_modules:BM840-1-BM840, symbol BM840
- removed U7: BT840, Fanstel_modules:BT840-BT840, symbol BT840
- added U?: BC832-V0, BC832_BC832, symbol BC832-V0
- added U?: BC832-V1, BC832_BC832, symbol BC832-V1
- added U?: BM832, BM832-1_BM832, symbol BM832
- added U?: BM840, BM840-1_BM840, symbol BM840
- added U?: BT840, BT840_BT840, symbol BT840
- added U?: BT832L, BT832_BT832L, symbol BT832L
- added U?: BT832X, BT832X_BT832X, symbol BT832X
Changed lines of the file:
@@
 EESchema Schematic File Version 2
+LIBS:Fanstel-modules
 LIBS:power
 LIBS:device
@@
 LIBS:contrib
 LIBS:valves
-LIBS:Fanstel-modules
 LIBS:Fanstel-kicad-library-cache
 EELAYER 25 0
@@
 Sheet 1 1
 Title ""
-Date "2018-07-11"
+Date "2018-07-15"
 Rev ""
 Comp ""
@@
 Comment4 ""
 $EndDescr
-Text Notes 2450 1100 0    60   ~ 0
+Text Notes 2150 1150 0    118  ~ 0
 BC832-V0
-Text Notes 5250 1100 0    60   ~ 0
+Text Notes 5100 1150 0    118  ~ 0
 BC832-V1
-Text Notes 8650 1100 0    60   ~ 0
+Text Notes 8650 1100 0    118  ~ 0
 BM832
-Text Notes 12450 1100 0    60   ~ 0
+Text Notes 12700 1100 0    118  ~ 0
 BM840
-Text Notes 3750 6000 0    60   ~ 0
+Text Notes 3550 6100 0    118  ~ 0
 BT832L
-Text Notes 7200 6050 0    60   ~ 0
+Text Notes 7600 6200 0    118  ~ 0
 BT832X
-Text Notes 11850 6050 0    60   ~ 0
+Text Notes 12600 6150 0    118  ~ 0
 BT840
 $Comp
-L BC832-V0 U1
-U 1 1 5B45F739
-P 2700 2250
-F 0 "U1" H 2700 2250 45  0001 C CNN
-F 1 "BC832-V0" H 2700 2250 45  0001 C CNN
-F 2 "Fanstel_modules:BC832-BC832" H 2730 2400 20  0001 C CNN
-F 3 "" H 2700 2250 60  0001 C CNN
-	1    2700 2250
+L BC832-V0 U?
+U 1 1 5B4AFE70
+P 2650 2450
+F 0 "U?" H 2650 3550 45  0000 C CNN
+F 1 "BC832-V0" H 3850 1600 45  0000 C CNN
+F 2 "BC832_BC832" H 2680 2600 20  0001 C CNN
+F 3 "" H 2650 2450 60  0001 C CNN
+	1    2650 2450
 	1    0    0    -1
 $EndComp
 $Comp
-L BC832-V1 U3
-U 1 1 5B45F74E
-P 5550 2200
-F 0 "U3" H 5550 2200 45  0001 C CNN
-F 1 "BC832-V1" H 5550 2200 45  0001 C CNN
-F 2 "Fanstel_modules:BC832-BC832" H 5580 2350 20  0001 C CNN
-F 3 "" H 5550 2200 60  0001 C CNN
-	1    5550 2200
+L BC832-V1 U?
+U 1 1 5B4B17E8
+P 5550 2450
+F 0 "U?" H 5550 3600 45  0000 C CNN
+F 1 "BC832-V1" H 6750 1550 45  0000 C CNN
+F 2 "BC832_BC832" H 5580 2600 20  0001 C CNN
+F 3 "" H 5550 2450 60  0001 C CNN
+	1    5550 2450
 	1    0    0    -1
 $EndComp
 $Comp
-L BM832 U4
-U 1 1 5B45F763
-P 7300 4400
-F 0 "U4" H 7300 4400 45  0001 C CNN
-F 1 "BM832" H 7300 4400 45  0001 C CNN
-F 2 "Fanstel_modules:BM832-1-BM832" H 7330 4550 20  0001 C CNN
-F 3 "" H 7300 4400 60  0001 C CNN
-	1    7300 4400
+L BM832 U?
+U 1 1 5B4B4B54
+P 8750 3000
+F 0 "U?" H 8850 4700 45  0000 C CNN
+F 1 "BM832" H 10200 1400 45  0000 C CNN
+F 2 "BM832-1_BM832" H 8750 3000 20  0001 C CNN
+F 3 "" H 7350 1450 60  0001 C CNN
+	1    8750 3000
 	1    0    0    -1
 $EndComp
 $Comp
-L BM840 U6
-U 1 1 5B45F778
-P 11250 4400
-F 0 "U6" H 11250 4400 45  0001 C CNN
-F 1 "BM840" H 11250 4400 45  0001 C CNN
-F 2 "Fanstel_modules:BM840-1-BM840" H 11280 4550 20  0001 C CNN
-F 3 "" H 11250 4400 60  0001 C CNN
-	1    11250 4400
+L BM840 U?
+U 1 1 5B4BB0C2
+P 13150 3150
+F 0 "U?" H 13100 4900 45  0000 C CNN
+F 1 "BM840" H 14500 1600 45  0000 C CNN
+F 2 "BM840-1_BM840" H 13150 3800 20  0001 C CNN
+F 3 "" H 11700 1650 60  0001 C CNN
+	1    13150 3150
 	1    0    0    -1
 $EndComp
 $Comp
-L BT832L U2
-U 1 1 5B45F78D
-P 4000 7050
-F 0 "U2" H 4000 7050 45  0001 C CNN
-F 1 "BT832L" H 4000 7050 45  0001 C CNN
-F 2 "Fanstel_modules:BT832-BT832L" H 4030 7200 20  0001 C CNN
-F 3 "" H 4000 7050 60  0001 C CNN
-	1    4000 7050
+L BT840 U?
+U 1 1 5B4C58AF
+P 12850 8300
+F 0 "U?" H 12850 10200 45  0000 C CNN
+F 1 "BT840" H 15300 7250 45  0000 C CNN
+F 2 "BT840_BT840" H 12680 8450 20  0001 C CNN
+F 3 "" H 12650 8300 60  0001 C CNN
+	1    12850 8300
 	1    0    0    -1
 $EndComp
 $Comp
-L BT832X U5
-U 1 1 5B45F7A9
-P 7450 8000
-F 0 "U5" H 7450 8000 45  0001 C CNN
-F 1 "BT832X" H 7450 8000 45  0001 C CNN
-F 2 "Fanstel_modules:BT832X-BT832X" H 7480 8150 20  0001 C CNN
-F 3 "" H 7450 8000 60  0001 C CNN
-	1    7450 8000
+L BT832L U?
+U 1 1 5B4C594A
+P 3900 7300
+F 0 "U?" H 3750 8300 45  0000 C CNN
+F 1 "BT832L" H 5250 6250 45  0000 C CNN
+F 2 "BT832_BT832L" H 3980 7450 20  0001 C CNN
+F 3 "" H 3950 7300 60  0001 C CNN
+	1    3900 7300
 	1    0    0    -1
 $EndComp
 $Comp
-L BT840 U7
-U 1 1 5B45F7CF
-P 11800 8050
-F 0 "U7" H 11800 8050 45  0001 C CNN
-F 1 "BT840" H 11800 8050 45  0001 C CNN
-F 2 "Fanstel_modules:BT840-BT840" H 11830 8200 20  0001 C CNN
-F 3 "" H 11800 8050 60  0001 C CNN
-	1    11800 8050
+L BT832X U?
+U 1 1 5B4C5C94
+P 7900 8300
+F 0 "U?" H 7900 10200 45  0000 C CNN
+F 1 "BT832X" H 9200 7300 45  0000 C CNN
+F 2 "BT832X_BT832X" H 7980 8400 20  0001 C CNN
+F 3 "" H 7950 8250 60  0001 C CNN
+	1    7900 8300
 	1    0    0    -1
 $EndComp
